File: hardware/Smoothiepanel/Smoothiepanel.brd (EAGLE design)
At the start: 119.4 x 72.4 mm, 75 parts, among them Q1 BC857B, U1 LPC11U24FBD64, U2 LM1117-3.3V, U3 MCP4725, X1 USB-B, X2 mUSB, X3 USB-MICROB-SMDRECEPT, X4 uSD, X5 SD, X6 VIN, Y1 12MHz

Commit message: Initial hardware commit (Prototype 5)
Parts:
- removed JP7: EXT, SparkFun-Connectors:1X05
- removed JP8: CHAR_LCD, logxen:TEXT_LCD
- removed U$11, U$8, U$9: MOUNTINGHOLE3.0THIN, microbuilder:MOUNTINGHOLE_3.0_PLATEDTHIN
- removed U$4, U$5, U$6, U$7: MOUNTINGHOLE2.5_THICK, microbuilder:MOUNTINGHOLE_2.5_PLATED_THICK
- removed X6: VIN, con-weidmueller-sl35:180-2
- added C17: 0.1uF, SparkFun-Capacitors:0603-CAP
- added C18, C19: 18pF, SparkFun-Capacitors:0603-CAP
- added JTAG1: JTAG, microbuilder:2X05_1.27MM_SMT
- added L1: FB, SparkFun-Passives:0603
- added LED1: POWER, SparkFun-LED:LED-0603
- added LED2: STATUS, SparkFun-LED:LED-0603
- added MH1, MH2, MH3, MH4, MH5, MH6, MH7: MOUNTINGHOLE2.5_THICK, microbuilder:MOUNTINGHOLE_2.5_PLATED_THICK
- added MH11, MH8, MH9: MOUNTINGHOLE3.0THIN, microbuilder:MOUNTINGHOLE_3.0_PLATEDTHIN
- added N1: NET_LINK, logxen:NET_LINK
- added R19: 33R, microbuilder:_0603MP
- added R20, R21: 0R, SparkFun-Passives:0603-RES
- added S3: BOOT, SparkFun-Electromechanical:TACTILE_SWITCH_SMD
- added SJ3: PSB, SparkFun:SJ_3
- added SJ4: VUART, SparkFun:SJ_3
- added SJ5: VSPI, SparkFun:SJ_3
- added SJ6: VDAC, SparkFun:SJ_3
- added SJ7: DAC_SCL, SparkFun-Passives:SJ_2S-TRACE
- added SJ8: DAC_SDA, SparkFun-Passives:SJ_2S-TRACE
- added TP1, TP3, TP4, TP5, TP6: TPAD1.5, logxen:TPAD-1.5
- added W3: WING3, logxen:PAPILIO-WING-8BITS-F
- added W4: WING4, logxen:PAPILIO-WING-8BITS-F
- added W5: WING5, logxen:PAPILIO-WING-8BITS-F
- added Z1: VIN, con-weidmueller-sl35:180-2
- added Z2: SYS_GND, logxen:1X03
- C1: value 0.1uF -> 1uF; device SparkFun-Capacitors:0603-CAP -> resistor:C0805
- C11: value 1uF -> 10uF; device resistor:C0805 -> SparkFun:EIA3216
- C12: value 10uF -> 0.1uF; device SparkFun:EIA3216 -> SparkFun-Capacitors:0603-CAP
- C14: value 0.1uF -> 18pF; device SparkFun-Capacitors:0603-CAP -> SparkFun-Passives:0603-CAP
- C15: device SparkFun-Capacitors:0603-CAP -> SparkFun-Passives:0603-CAP
- C16, C3, C4: value 18pF -> 0.1uF
- JP1: value LCD -> VIN; device logxen:1X22 -> con-amp:10X02MTA
- JP2: value VIN -> SYS; device con-amp:10X02MTA -> logxen:1X03
- JP3: value SPI0 -> GLCD; device SparkFun-Connectors:2X3-SHROUDED -> logxen:1X22
- JP4: device SparkFun-Connectors:1X06 -> logxen:1X06
- JP5: value SPI1/SD -> SPI0; device SparkFun-Connectors:2X3-SHROUDED -> logxen:2X3-SHROUDED
- JP6: value I2C -> CHAR_LCD; device SparkFun-Connectors:1X05 -> logxen:TEXT_LCD
- R1: value 0R -> 330R
- R10: value 100 Ohm -> 0R
- R11: value 10kOhm -> 0R
- R12: device SparkFun-Resistors:0603-RES -> SparkFun-Passives:0603-RES
- R13, R14, R3, R4: value 10kOhm -> 10K
- R15: value 10kOhm -> 3K
- R16: value 0R -> 33R; device resistor:R0603 -> microbuilder:_0603MP
- R17: value 0R -> 24K; device resistor:R0603 -> SparkFun-Resistors:0603-RES
- R18: device resistor:R0603 -> SparkFun-Passives:0603-RES
- R2: value 1.5kOhm -> 10K
- R22: value 0R -> 100R
- R23: value 0R -> 1.5K
- R24: value 0R -> NP
- R5: value 10kOhm -> 330R
- R6: value 33 Ohm -> 0R
- R7: value 33 Ohm -> 10K
- R8: value 3kOhm -> 10K
- R9: value 24kOhm -> 10K
- SJ1: value VUART -> GLCDV
- SJ2: device SparkFun-Passives:SJ_3_PASTE2&3 -> SparkFun-Passives:SJ_3
- U1: value LPC11U24FBD64 -> LM1117-3.3V; device microbuilder:LQFP64 -> SparkFun:SOT223
- U2: value LM1117-3.3V -> LPC176xFBD100; device SparkFun:SOT223 -> microbuilder:LQFP100
- W1: value PAPILIO-WING-8BITS -> WING1; device logxen:PAPILIO-WING-8BITS -> logxen:PAPILIO-WING-8BITS-F
- W2: value PAPILIO-WING-8BITS -> WING2; device logxen:PAPILIO-WING-8BITS -> logxen:PAPILIO-WING-8BITS-F
- X4: value uSD -> SD; device SparkFun-Connectors:MICRO-SD-SOCKET-PP -> SparkFun-Connectors:SDCARD_4UCONN
- X5: value SD -> uSD; device SparkFun-Connectors:SDCARD_4UCONN -> SparkFun-Connectors:MICRO-SD-SOCKET-PP
- Y1: device microbuilder:CRYSTAL_2.5X2 -> microbuilder:CRYSTAL_3.2X2.5
- moved JP6 100.6 mm to (24.1, 69.8), turned to 0 degrees
- moved R18 96.3 mm to (67.3, 64.8), turned to 270 degrees
- moved R3 84.3 mm to (15.2, 29.2), turned to 0 degrees
- moved JP3 79.5 mm to (76.2, 5.08), turned to 180 degrees
- moved R23 78.8 mm to (17.5, 58.7)
- moved C13 77.2 mm to (98.7, 13.0)
- moved R22 73.6 mm to (21.3, 51.8), turned to 180 degrees
- moved R16 72.2 mm to (38.1, 48.6), turned to 135 degrees
- moved R11 70.5 mm to (27.9, 9.84), turned to 90 degrees
- moved R17 69.6 mm to (22.9, 54.6), turned to 90 degrees
- moved C1 66.7 mm to (90.5, 38.7), turned to 0 degrees
- moved C9 65.4 mm to (38.7, 38.7), turned to 270 degrees
- moved SJ1 65.2 mm to (81.3, 5.08), turned to 180 degrees
- moved C10 65.0 mm to (90.5, 41.0), turned to 0 degrees
- moved R9 60.9 mm to (83.8, 40.0), turned to 270 degrees
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- renumbered U$10 to MH10
Connections:
- removed net DAC_SCL: JP7.3, U1.23, U3.5
- removed net DAC_SDA: JP7.4, U1.63, U3.4
- removed net MISO: JP3.4, U1.36
- removed net MOSI: JP3.6, U1.37
- removed net P0_11: U1.42, W1.1
- removed net P0_12: U1.44, W1.2
- removed net P0_13: U1.45, W1.3
- removed net P0_14: U1.46, W1.4
- removed net P0_15: U1.52, W1.5
- removed net P0_16: U1.53, W1.6
- removed net P0_23: U1.56, W1.8
- removed net P1_11: U1.43, W2.4
- removed net P1_12: U1.59, W2.5
- removed net P1_13: U1.47, W2.6
- removed net RXD: JP4.4, U1.61
- removed net SCK: JP3.5, U1.41
- removed net SCL: JP6.4, PCB1.3, R11.1, U1.20
- removed net SDA: JP6.3, PCB1.6, R3.1, U1.21
- removed net SD_MISO: JP5.4, R14.1, U1.35, X4.7, X5.7
- removed net SD_MOSI: JP5.6, R15.1, U1.51, X4.3, X5.2
- removed net SD_SCK: JP5.5, U1.18, X4.5, X5.5
- removed net SD_SSEL: JP7.5, R13.1, U1.30, X4.2, X5.1
- removed net SSEL: JP3.3, U1.13
- removed net TXD: JP4.5, U1.62
- removed net VO: JP8.VO
- removed net XTALIN: C15.2, U1.8, Y1.1
- removed net XTALOUT: C16.2, U1.9, Y1.3
- new net !RSTOUT!: U2.14
- new net !TRST!: JTAG1.10, U2.4
- new net ADC0: U2.9, W1.1
- new net ADC1: U2.8, W1.2
- new net ADC2: U2.7, W1.3
- new net ADC3: U2.6, W1.4
- new net AGND: C16.2, N1.P$1, U2.11, U2.15
- new net AVCC: C16.1, L1.1, U2.10, U2.12
- new net DAC_SCL_RES: SJ7.2, U3.5
- new net DAC_SDA_RES: SJ8.2, U3.4
- new net DAC_VIN: SJ6.2, U3.3
- new net LCD_V: C2.1, C3.1, JP3.19, JP3.2, JP6.A, JP6.VDD, SJ1.2
- new net LED1_R: LED1.A, R1.2
- new net LED2_R: LED2.A, R5.2
- new net MISO0: JP5.6, U2.61
- new net MISO1: R7.1, U2.77, W3.7, X4.7, X5.7
- new net MOSI0: JP5.4, U2.60
- new net MOSI1: R8.1, U2.76, W3.8, X4.2, X5.3
- new net P0_19: U2.59, W2.4
- new net P0_20: U2.58, W2.3
- new net P0_21: U2.57, W2.2
- new net P0_4: U2.81, W2.5
- new net P0_5: LED2.C, U2.80, W2.8
- new net P1_0: U2.95, W5.8
- new net P1_1: U2.94, W5.7
- new net P1_16: U2.87, W4.8
- new net P1_17: U2.86, W4.7
- new net P1_21: U2.35, W1.7
- new net P1_22: U2.36, W1.8
- new net P1_4: U2.93, W5.6
- new net PCAP0: U2.44, W4.5
- new net PCAP1: U2.45, W4.6
- new net PHA: U2.34, W1.5
- new net PHB: U2.37, W1.6
- new net PWM5: U2.38, W4.3
- new net PWM6: U2.40, W4.4
- new net RXD0: JP4.4, U2.99
- new net RXD2: U2.49, W4.2
- new net RXD3: U2.85, W3.2
- new net SCK0: JP5.5, U2.62
- new net SCK1: U2.78, W3.6, X4.5, X5.5
- new net SCL0: PCB1.3, R13.1, U2.24, W3.3
- new net SCL1: SJ7.1, U2.47, W2.6
- new net SDA0: PCB1.6, R14.1, U2.25, W3.4
- new net SDA1: SJ8.1, U2.46, W2.7
- new net SSEL0: JP5.3, U2.63
- new net SSEL1_A: U2.65, W3.5
- new net TCK: JTAG1.4, U2.5
- new net TDI: JTAG1.8, U2.2
- new net TDO: JTAG1.6, U2.1
- new net TMS: JTAG1.2, U2.3
- new net TXD0: JP4.5, U2.98
- new net TXD2: U2.48, W4.1
- new net TXD3: U2.82, W3.1
- new net VSPI: JP5.1, SJ5.2
- new net XTAL1: C14.1, U2.22, Y1.2
- new net XTAL2: C15.1, U2.23, Y1.1
- net 3.3V: now also C10.1, C12.1, C4.1, C9.1, JTAG1.1, L1.2, R1.1, R17.2, R2.2, R3.2, R5.1, R7.2, R8.2, SJ3.1, SJ4.3, SJ5.3, U1.2, U1.4, U2.19, U2.28, U2.42, U2.54, U2.71, U2.84, U2.96, W3.11, W4.11, W5.11; no longer C11.1, C13.1, C14.1, C2.1, JP1.19, JP1.2, JP3.1, JP5.1, JP7.1, JP8.A, PCB1.4, R13.2, R14.2, R15.2, R5.2, U1.10, U1.33, U1.48, U1.58, U2.2, U2.4
- net 5V: now also C11.A, SJ4.1, SJ5.1, SJ6.1, U1.3, W3.12, W4.12, W5.12; no longer C12.A, JP8.VDD, U2.3
- net DM: now also R19.2; no longer R6.2
- net DP: now also R16.2, R23.2; no longer R2.2, R7.2
- net GND: now also C11.C, C12.2, C15.2, C17.2, C18.2, C19.2, JP1.2, JP3.1, JP6.GND, JTAG1.3, JTAG1.5, JTAG1.9, LED1.C, N1.P$2, R24.1, S3.1, S3.2, SJ3.3, U1.1, U2.31, U2.41, U2.55, U2.72, U2.83, U2.97, W3.9, W4.9, W5.9, X4.3, X4.SH@1, X4.SH@2, X5.GND1, X5.GND3, Z1.2, Z2.1, Z2.2, Z2.3; no longer C11.2, C12.C, C15.1, C16.1, JP1.1, JP2.2, JP3.2, JP6.2, JP7.2, JP8.GND, R1.1, U1.54, U1.7, U2.1, X4.CD2, X4.GND1, X4.GND3, X5.3, X5.SH@1, X5.SH@2, X6.2
- net INT: now also TP4.1, U2.52; no longer JP6.5, U1.22
- net ISP: now also JP2.2, R3.1, U2.53; no longer R5.1, U1.5
- net LCD_D0: now also JP3.7, JP6.D0, U2.75; no longer JP1.7, U1.1
- net LCD_D1: now also JP3.8, JP6.D1, U2.74; no longer JP1.8, U1.17
- net LCD_D2: now also JP3.9, JP6.D2, U2.73; no longer JP1.9, U1.34
- net LCD_D3: now also JP3.10, JP6.D3, U2.70; no longer JP1.10, U1.50
- net LCD_D4: now also JP3.11, JP6.D4, U2.69; no longer JP1.11, JP8.D4, U1.16
- net LCD_D5: now also JP3.12, JP6.D5, U2.68; no longer JP1.12, JP8.D5, U1.32
- net LCD_D6: now also JP3.13, JP6.D6, U2.67; no longer JP1.13, JP8.D6, U1.64
- net LCD_D7: now also JP3.14, JP6.D7, U2.66; no longer JP1.14, JP8.D7, U1.6
- net LCD_EN: now also JP3.6, JP6.E, U2.43; no longer JP1.6, JP8.E, U1.11
- net LCD_LEDB: now also R18.2, R6.2, U2.26; no longer R16.2, R22.2, U1.14
- net LCD_LEDB_RES: now also JP3.22, R6.1; no longer JP1.22, R22.1
- net LCD_LEDB_RES1: now also JP6.B, R18.1; no longer JP8.B, R16.1
- net LCD_LEDG: now also R10.2, R20.2, U2.27; no longer R17.2, R23.2, U1.2
- net LCD_LEDG_RES: now also JP3.21, R10.1; no longer JP1.21, R23.1
- net LCD_LEDG_RES1: now also JP6.G, R20.1; no longer JP8.G, R17.1
- net LCD_LEDR: now also R11.2, R21.2, U2.32; no longer R18.2, R24.2, U1.27
- net LCD_LEDR_RES: now also JP3.20, R11.1; no longer JP1.20, R24.1
- net LCD_LEDR_RES1: now also JP6.R, R21.1; no longer JP8.R, R18.1
- net LCD_PSB: now also JP3.15, SJ3.2; no longer JP1.15, U1.31
- net LCD_R/W: now also JP3.5, JP6.R/W, U2.33; no longer JP1.5, JP8.R/W, U1.38
- net LCD_RS: now also JP3.4, JP6.RS, U2.39; no longer JP1.4, JP8.RS, U1.60
- net LCD_RST: now also JP2.3, JP3.17, R4.1, S3.3, S3.4, U2.20; no longer JP1.17, U1.15
- net LCD_VO: now also C17.1, JP3.3, JP6.VO, R24.2; no longer C10.1, JP1.3, R1.2
- net LCD_VOUT: now also JP3.18, SJ6.3; no longer JP1.18, U3.3
- net P0_22: now also U2.56, W2.1; no longer U1.40, W1.7
- net P1_10: now also U2.90, W5.3; no longer U1.12, W2.3
- net P1_14: now also U2.89, W5.2; no longer U1.49, W2.7
- net P1_15: now also U2.88, W5.1; no longer U1.57, W2.8
- net P1_8: now also U2.92, W5.5; no longer U1.39, W2.1
- net P1_9: now also U2.91, W5.4; no longer U1.55, W2.2
- net RESET: now also JP2.1, R2.1, U2.17; no longer R4.1, U1.4
- net SD_CD: now also TP5.1, U2.51, X4.CD, X5.CD1, X5.CD2; no longer U1.28, X4.CD1, X5.CD
- net SD_WP: now also TP6.1, U2.50, X4.WP; no longer U1.3, X5.WP
- net SSEL1: now also R9.1, U2.79, X4.1, X5.2; no longer JP5.3, U1.24
- net USB_CONNECT: now also R15.1, TP3.1, U2.64; no longer R8.1, U1.29
- net USB_CONNECT_BASE: now also R15.2, R17.1; no longer R8.2, R9.1
- net USB_CONNECT_COLLECTOR: now also R23.1; no longer R2.1
- net USB_DM: now also C19.1, R19.1, U2.30; no longer C4.1, R6.1, U1.25
- net USB_DP: now also C18.1, R16.1, U2.29; no longer C3.1, R7.1, U1.26
- net USB_VBUS: now also R22.1, TP1.1, U2.21; no longer R10.1, U1.19
- net VBUS: now also R22.2; no longer R10.2
- net VI2C: now also C13.1, PCB1.4, R13.2, R14.2; no longer C9.1, JP6.1, R11.2, R3.2
- net VIN: now also JP1.1, Z1.1; no longer JP2.1, X6.1
- net VUART: now also SJ4.2; no longer SJ1.2
Routing:
- net 3.3V: track 511.7 -> 156.0 mm, vias 17 -> 24
- net LCD_V: track 0.00 -> 205.2 mm, vias 0 -> 2
- net SDA0: track 0.00 -> 148.8 mm, vias 0 -> 4
- net SCL0: track 0.00 -> 143.7 mm, vias 0 -> 3
- net LCD_R/W: track 35.0 -> 176.3 mm, vias 1 -> 4
- net LCD_RS: track 37.8 -> 176.3 mm, vias 2 -> 4
- net P0_5: track 0.00 -> 133.8 mm, vias 0 -> 3
- net LCD_LEDG: track 24.7 -> 154.9 mm, vias 2 -> 4
- net GND: track 238.0 -> 111.0 mm, vias 32 -> 103
- net LCD_LEDB: track 32.8 -> 152.8 mm
- net LCD_VO: track 13.7 -> 133.2 mm, vias 0 -> 2
- net LCD_EN: track 48.1 -> 167.3 mm, vias 2 -> 4
- net LCD_D6: track 18.7 -> 136.0 mm, vias 0 -> 2
- net LCD_D3: track 19.7 -> 136.7 mm
- net LCD_LEDR: track 41.3 -> 153.3 mm, vias 2 -> 4
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- added copper zone on layer 15, net 3.3V
- added copper zone on layer 2, net GND
- added copper zone on layer 1, net MCU_KEEPOUT
Other:
- board size 119.4 x 72.4 mm -> 124.5 x 73.7 mm
- board text added: "0.0(SDA1)"
- board text added: "0.0(SDA1) 1.10"
- board text added: "0.1(SCL1)"
- board text added: "0.1(SCL1) 1.14"
- board text added: "0.10 1.20"
- board text added: "0.11 1.23"
- board text added: "0.15 SCK"
- board text added: "0.16 SSEL"
- board text added: "0.17 MISO"
- board text added: "0.18 MOSI"
- board text added: "0.19 1.16"
- board text added: "0.2 TXD"
- board text added: "0.20 1.17"
- board text added: "0.21 1.29"
- board text added: "0.22 1.28"
- board text added: "0.23(ADC0)"
- board text added: "0.24(ADC1)"
- board text added: "0.25(ADC2)"
- board text added: "0.26(ADC3)"
- board text added: "0.27 0.28 2.11"
- board text added: "0.27(SDA0) 1.0"
- board text added: "0.28(SCL0) 1.1"
- board text added: "0.3 RXD"
- board text added: "0.4 1.15"
- board text added: "0.5(LED) 1.9"
- board text added: "0.6(SSEL1)"
- board text added: "0.7(SCK1)"
- board text added: "0.8(MISO1)"
- board text added: "0.9(MOSI1)"
- board text added: "1.0 0.27(SDA0)"
- board text added: "1.1 0.28(SCL0)"
- board text added: "1.10"
- board text added: "1.14"
- board text added: "1.15 0.4"
- board text added: "1.16 0.19"
- board text added: "1.17 0.20"
- board text added: "1.20 0.10"
- board text added: "1.21 1.24"
- board text added: "1.22 1.26"
- board text added: "1.23 0.11"
- board text added: "1.24 1.21"
- board text added: "1.26 1.22"
- board text added: "1.28 0.22"
- board text added: "1.29 0.21"
- board text added: "1.4 4.29(RXD3)"
- board text added: "1.8 4.28(TXD3)"
- board text added: "1.9 0.5(LED)"
- board text added: "4.28(TXD3) 1.8"
- board text added: "4.29(RXD3) 1.4"
- board text added: "B- 3.26"
- board text added: "BOOT"
- board text added: "BOOT 1.31"
- board text added: "CHAR LCD"
- board text added: "D0 2.0"
- board text added: "D1 2.1"
- board text added: "D2 2.2"
- board text added: "D3 2.3"
- board text added: "D4 2.4"
- board text added: "D5 2.5"
- board text added: "D6 2.6"
- board text added: "D7 2.7"
- board text added: "EN 1.27"
- board text added: "G- 3.25"
- board text added: "GLCD"
- board text added: "ISP"
- board text added: "ISP 2.10"
- board text added: "JP3"
- board text added: "POWER"
- board text added: "Prototype 5"
- board text added: "R- 1.18"
- board text added: "R/W 1.19"
- board text added: "RS 1.25"
- board text added: "RST 1.31"
- board text added: "SDA0 SCL0 INT"
- board text added: "STATUS"
- board text added: "V+"
- board text added: "VDAC"
- board text added: "VLCD"
- board text added: "VSPI"
- board text removed: "... P0.16"
- board text removed: "... P1.15"
- board text removed: "/INT"
- board text removed: "EXT"
- board text removed: "I2C"
- board text removed: "INT"
- board text removed: "JP7"
- board text removed: "LCD"
- board text removed: "P0.11 ..."
- board text removed: "P0.22"
- board text removed: "P0.23"
- board text removed: "P0.7/SD_SSEL"
- board text removed: "P1.16/DAC_SDA"
- board text removed: "P1.17/DAC_SCL"
- board text removed: "P1.8 ..."
- board text removed: "Prototype 3"
- board text removed: "SCL"
- board text removed: "SDA"
- board text removed: "SPI PINOUT"
- board text removed: "SPI1"
- board text removed: "W1"
- board text removed: "W2"
- board text removed: "uUSB"
