File: hardware/Smoothiepanel/Smoothiepanel.sch (EAGLE design)
At the start: 73 parts, among them Q1 BC857B, U1 LPC11U24FBD64, U2 LM1117-3.3V, U3 MCP4725, X1 USB-B, X2 mUSB, X3 USB-MICROB-SMDRECEPT, X4 uSD, X5 SD, X6 VIN, Y1 12MHz

Commit message: Initial hardware commit (Prototype 5)
Parts:
- removed JP7: EXT, SparkFun-Connectors:M05PTH
- removed JP8: CHAR_LCD, logxen:LCD_TEXT
- removed U$10, U$11, U$8, U$9: MOUNTINGHOLE3.0THIN, microbuilder:MOUNTINGHOLE3.0THIN
- removed U$4, U$5, U$6, U$7: MOUNTINGHOLE2.5_THICK, microbuilder:MOUNTINGHOLE2.5_THICK
- removed X6: VIN, con-weidmueller-sl35:180-2
- added C17: 0.1uF, SparkFun-Capacitors:CAP0603-CAP
- added C18, C19: 18pF, SparkFun-Capacitors:CAP0603-CAP
- added JTAG1: JTAG, microbuilder:JTAG-CORTEXM3
- added L1: FB, SparkFun-Passives:INDUCTOR0603
- added LED1: POWER, SparkFun-LED:LED0603
- added LED2: STATUS, SparkFun-LED:LED0603
- added MH1, MH2, MH3, MH4, MH5, MH6, MH7: MOUNTINGHOLE2.5_THICK, microbuilder:MOUNTINGHOLE2.5_THICK
- added MH10, MH11, MH8, MH9: MOUNTINGHOLE3.0THIN, microbuilder:MOUNTINGHOLE3.0THIN
- added N1: NET_LINK, logxen:NET_LINK
- added R19: 33R, microbuilder:RESISTOR_0603MP
- added R20, R21: 0R, SparkFun-Passives:RESISTOR0603-RES
- added S3: BOOT, SparkFun-Electromechanical:TAC_SWITCHSMD
- added SJ3: PSB, SparkFun:SOLDERJUMPER_2WAYS
- added SJ4: VUART, SparkFun:SOLDERJUMPER_2WAYS
- added SJ5: VSPI, SparkFun:SOLDERJUMPER_2WAYS
- added SJ6: VDAC, SparkFun:SOLDERJUMPER_2WAYS
- added SJ7: DAC_SCL, SparkFun-Passives:SOLDERJUMPERTRACE
- added SJ8: DAC_SDA, SparkFun-Passives:SOLDERJUMPERTRACE
- added TP1, TP3, TP4, TP5, TP6: TPAD1.5, logxen:TPAD1.5
- added W3: WING3, logxen:PAPILIO-WING-8BITSF
- added W4: WING4, logxen:PAPILIO-WING-8BITSF
- added W5: WING5, logxen:PAPILIO-WING-8BITSF
- added Z1: VIN, con-weidmueller-sl35:180-2
- added Z2: SYS_GND, logxen:M03PTH
- C1: value 0.1uF -> 1uF; device SparkFun-Capacitors:CAP0603-CAP -> resistor:C-USC0805
- C11: value 1uF -> 10uF; device resistor:C-USC0805 -> SparkFun:CAP_POL1206
- C12: value 10uF -> 0.1uF; device SparkFun:CAP_POL1206 -> SparkFun-Capacitors:CAP0603-CAP
- C14: value 0.1uF -> 18pF; device SparkFun-Capacitors:CAP0603-CAP -> SparkFun-Passives:CAP0603-CAP
- C15: device SparkFun-Capacitors:CAP0603-CAP -> SparkFun-Passives:CAP0603-CAP
- C16, C3, C4: value 18pF -> 0.1uF
- JP1: value LCD -> VIN; device logxen:M22 -> con-amp:MTA02-100
- JP2: value VIN -> SYS; device con-amp:MTA02-100 -> logxen:M03PTH
- JP3: value SPI0 -> GLCD; device SparkFun-Connectors:M03X2 -> logxen:M22
- JP4: device SparkFun-Connectors:M06SIP -> logxen:M06SIP
- JP5: value SPI1/SD -> SPI0; device SparkFun-Connectors:M03X2 -> logxen:M03X2
- JP6: value I2C -> CHAR_LCD; device SparkFun-Connectors:M05PTH -> logxen:LCD_TEXT
- R1: value 0R -> 330R
- R10: value 100 Ohm -> 0R
- R11: value 10kOhm -> 0R
- R12: device SparkFun-Resistors:RESISTOR0603-RES -> SparkFun-Passives:RESISTOR0603-RES
- R13, R14, R3, R4: value 10kOhm -> 10K
- R15: value 10kOhm -> 3K
- R16: value 0R -> 33R; device resistor:R-US_R0603 -> microbuilder:RESISTOR_0603MP
- R17: value 0R -> 24K; device resistor:R-US_R0603 -> SparkFun-Resistors:RESISTOR0603-RES
- R18: device resistor:R-US_R0603 -> SparkFun-Passives:RESISTOR0603-RES
- R2: value 1.5kOhm -> 10K
- R22: value 0R -> 100R
- R23: value 0R -> 1.5K
- R24: value 0R -> NP
- R5: value 10kOhm -> 330R
- R6: value 33 Ohm -> 0R
- R7: value 33 Ohm -> 10K
- R8: value 3kOhm -> 10K
- R9: value 24kOhm -> 10K
- SJ1: value VUART -> GLCDV
- SJ2: device SparkFun-Passives:SOLDERJUMPER_2WAYPASTE2&3 -> SparkFun-Passives:SOLDERJUMPER_2WAYS
- U1: value LPC11U24FBD64 -> LM1117-3.3V; device microbuilder:LPC11U24_QFP64 -> SparkFun:V_REG_LM1117SOT223
- U2: value LM1117-3.3V -> LPC176xFBD100; device SparkFun:V_REG_LM1117SOT223 -> microbuilder:LPC1768
- W1: value PAPILIO-WING-8BITS -> WING1; device logxen:PAPILIO-WING-8BITS -> logxen:PAPILIO-WING-8BITSF
- W2: value PAPILIO-WING-8BITS -> WING2; device logxen:PAPILIO-WING-8BITS -> logxen:PAPILIO-WING-8BITSF
- X4: value uSD -> SD; device SparkFun-Connectors:USD-SOCKETNEW -> SparkFun-Connectors:SD_CARD_SOCKET4UCON
- X5: value SD -> uSD; device SparkFun-Connectors:SD_CARD_SOCKET4UCON -> SparkFun-Connectors:USD-SOCKETNEW
- Y1: device microbuilder:CRYSTAL2.5X2.0MM -> microbuilder:CRYSTALTHIN
Connections:
- removed net DAC_SCL: JP7.3, U1.PIO1_17/CT16B0_CAP1/RXD, U3.SCL
- removed net DAC_SDA: JP7.4, U1.PIO1_16/RI/CT16B0_CAP0, U3.SDA
- removed net MISO: JP3.4, U1.PIO0_8/MISO0/CT16B0_MAT0
- removed net MOSI: JP3.6, U1.PIO0_9/MOSI0/CT16B0_MAT1
- removed net P0_11: U1.TDI/PIO0_11/AD0/CT32B0_MAT3, W1.P1
- removed net P0_12: U1.TMS/PIO0_12/AD1/CT32B1_CAP0, W1.P2
- removed net P0_13: U1.TDO/PIO0_13/AD2/CT32B1_MAT0, W1.P3
- removed net P0_14: U1.TRST/PIO0_14/AD3/CT32B1_MAT1, W1.P4
- removed net P0_15: U1.SWDIO/PIO0_15/AD4/CT32B1_MAT2, W1.P5
- removed net P0_16: U1.PIO0_16/AD5/CT32B1_MAT3/WAKEUP, W1.P6
- removed net P0_23: U1.PIO0_23/AD7, W1.P8
- removed net P1_11: U1.PIO1_11, W2.P4
- removed net P1_12: U1.PIO1_12, W2.P5
- removed net P1_13: U1.PIO1_13/DTR/CT16B0_MAT0/TXD, W2.P6
- removed net RXD: JP4.4, U1.PIO0_18/RXD/CT32B0_MAT0
- removed net SCK: JP3.5, U1.PIO1_29/SCK0/CT32B0_CAP1
- removed net SCL: JP6.4, PCB1.SCL, R11.1, U1.PIO0_4/SCL-(20MA_SINK)
- removed net SDA: JP6.3, PCB1.SDA, R3.1, U1.PIO0_5/SDA-(20MA_SINK)
- removed net SD_MISO: JP5.4, R14.1, U1.PIO1_21/DCD/MISO1, X4.DO, X5.DAT0
- removed net SD_MOSI: JP5.6, R15.1, U1.PIO1_22/RI/MOSI1, X4.DI, X5.CMD
- removed net SD_SCK: JP5.5, U1.PIO1_20/DSR/SCK1, X4.SCK, X5.CLK
- removed net SD_SSEL: JP7.5, R13.1, U1.PIO0_7/CTS-(20MA_SOURCE), X4.CS, X5.CD/DAT3
- removed net SSEL: JP3.3, U1.PIO0_2/SSEL0/CT16B0_CAP0
- removed net TXD: JP4.5, U1.PIO0_19/TXD/CT32B0_MAT1
- removed net VO: JP8.3
- removed net XTALIN: C15.2, U1.XTALIN, Y1.1
- removed net XTALOUT: C16.2, U1.XTALOUT, Y1.2
- new net !RSTOUT!: U2.RSTOUT
- new net !TRST!: JTAG1.10, U2.TRST
- new net ADC0: U2.P0[23]/AD0[0]/I2SRX_CLK/CAP3[0], W1.P1
- new net ADC1: U2.P0[24]/AD0[1]/I2SRX_WS/CAP3[1], W1.P2
- new net ADC2: U2.P0[25]/AD0[2]/I2SRX_SDA/TXD3, W1.P3
- new net ADC3: U2.P0[26]/AD0[3]/AOUT/RXD3, W1.P4
- new net AGND: C16.2, N1.P$1, U2.VREFN, U2.VSSA
- new net AVCC: C16.1, L1.1, U2.VDDA, U2.VREFP
- new net DAC_SCL_RES: SJ7.2, U3.SCL
- new net DAC_SDA_RES: SJ8.2, U3.SDA
- new net DAC_VIN: SJ6.2, U3.VDD
- new net LCD_V: C2.1, C3.1, JP3.19, JP3.2, JP6.15, JP6.2, SJ1.2
- new net LED1_R: LED1.A, R1.2
- new net LED2_R: LED2.A, R5.2
- new net MISO0: JP5.6, U2.P0[17]/CTS1/MISO0/MISO
- new net MISO1: R7.1, U2.P0[8]/I2STX_WS/MISO1/MAT2[2], W3.P7, X4.DAT0, X5.DO
- new net MOSI0: JP5.4, U2.P0[18]/DCD1/MOSI0/MOSI
- new net MOSI1: R8.1, U2.P0[9]/I2STX_SDA/MOSI1/MAT2[3], W3.P8, X4.CMD, X5.DI
- new net P0_19: U2.P0[19]/DSR1/SDA1, W2.P4
- new net P0_20: U2.P0[20]/DTR1/SCL1, W2.P3
- new net P0_21: U2.P0[21]/RI1/RD1, W2.P2
- new net P0_4: U2.P0[4]/I2SRX_CLK/RD2/CAP2[0], W2.P5
- new net P0_5: LED2.C, U2.P0[5]/I2SRX_WS/TD2/CAP2[1], W2.P8
- new net P1_0: U2.P1[0]/ENET_TXD0, W5.P8
- new net P1_1: U2.P1[1]/ENET_TXD1, W5.P7
- new net P1_16: U2.P1[16]/ENET_MDC, W4.P8
- new net P1_17: U2.P1[17]/ENET_MDIO, W4.P7
- new net P1_21: U2.P1[21]/MCABORT/PWM1[3]/SSEL0, W1.P7
- new net P1_22: U2.P1[22]/MC0B/USB_PWRD/MAT1[0], W1.P8
- new net P1_4: U2.P1[4]/ENET_TX_EN, W5.P6
- new net PCAP0: U2.P1[28]/MC2A/PCAP1[0]/MAT0[0], W4.P5
- new net PCAP1: U2.P1[29]/MC2B/PCAP1[1]/MAT0[1], W4.P6
- new net PHA: U2.P1[20]/MCFB0/PWM1[2]/SCK0, W1.P5
- new net PHB: U2.P1[23]/MCFB1/PWM1[4]/MISO0, W1.P6
- new net PWM5: U2.P1[24]/MCFB2/PWM1[5]/MOSI0, W4.P3
- new net PWM6: U2.P1[26]/MC1B/PWM1[6]/CAP0[0], W4.P4
- new net RXD0: JP4.4, U2.P0[3]/RXD0/AD0[6]
- new net RXD2: U2.P0[11]/RXD2/SCL2/MAT3[1], W4.P2
- new net RXD3: U2.P4[29]/TX_MCLK/MAT2[1]/RXD3, W3.P2
- new net SCK0: JP5.5, U2.P0[15]/TXD1/SCK0/SCK
- new net SCK1: U2.P0[7]/I2STX_CLK/SCK1/MAT2[1], W3.P6, X4.CLK, X5.SCK
- new net SCL0: PCB1.SCL, R13.1, U2.P0[28]/SCL0/USB_SCL, W3.P3
- new net SCL1: SJ7.1, U2.P0[1]/TD1/RXD3/SCL1, W2.P6
- new net SDA0: PCB1.SDA, R14.1, U2.P0[27]/SDA0/USB_SDA, W3.P4
- new net SDA1: SJ8.1, U2.P0[0]/RD1/TXD3/SDA1, W2.P7
- new net SSEL0: JP5.3, U2.P0[16]/RXD1/SSEL0/SSEL
- new net SSEL1_A: U2.P2[8]/TD2/TXD2, W3.P5
- new net TCK: JTAG1.4, U2.TCK/SWDCLK
- new net TDI: JTAG1.8, U2.TDI
- new net TDO: JTAG1.6, U2.TDO/SWO
- new net TMS: JTAG1.2, U2.TMS/SWDIO
- new net TXD0: JP4.5, U2.P0[2]/TXD0/AD0[7]
- new net TXD2: U2.P0[10]/TXD2/SDA2/MAT3[0], W4.P1
- new net TXD3: U2.P4[28]/RX_MCLK/MAT2[0]/TXD3, W3.P1
- new net VSPI: JP5.1, SJ5.2
- new net XTAL1: C14.1, U2.XTAL1, Y1.2
- new net XTAL2: C15.1, U2.XTAL2, Y1.1
- net 3.3V: now also C10.1, C12.1, C4.1, C9.1, JTAG1.1, L1.2, R1.1, R17.2, R2.2, R3.2, R5.1, R7.2, R8.2, SJ3.1, SJ4.3, SJ5.3, U1.OUT, U1.OUT@1, U2.VBAT, U2.VDD(3V3)1, U2.VDD(3V3)2, U2.VDD(3V3)3, U2.VDD(3V3)4, U2.VDD(REG)(3V3)1, U2.VDD(REG)(3V3)2, W3.3.3V, W4.3.3V, W5.3.3V, X4.VDD, X5.VCC; no longer C11.1, C13.1, C14.1, C2.1, JP1.19, JP1.2, JP3.1, JP5.1, JP7.1, JP8.15, PCB1.VCC, R13.2, R14.2, R15.2, R5.2, U1.VDD@1, U1.VDD@2, U1.VDD@3, U1.VDD@4, U2.OUT, U2.OUT@1, X4.VCC, X5.VDD
- net 5V: now also C11.+, SJ4.1, SJ5.1, SJ6.1, U1.IN, W3.5V, W4.5V, W5.5V; no longer C12.+, JP8.2, U2.IN
- net DM: now also R19.2; no longer R6.2
- net DP: now also R16.2, R23.2; no longer R2.2, R7.2
- net GND: now also C11.-, C12.2, C15.2, C17.2, C18.2, C19.2, JP1.2, JP3.1, JP6.1, JTAG1.3, JTAG1.5, JTAG1.9, LED1.C, N1.P$2, R24.1, S3.1, S3.2, SJ3.3, U1.ADJ, U2.VSS1, U2.VSS2, U2.VSS3, U2.VSS4, U2.VSS5, U2.VSS6, W3.GND, W4.GND, W5.GND, X4.SH@1, X4.SH@2, X4.VSS1, X4.VSS2, X5.GND, X5.SHIELD@1, X5.SHIELD@3, Z1.2, Z2.1, Z2.2, Z2.3; no longer C11.2, C12.-, C15.1, C16.1, JP1.1, JP2.2, JP3.2, JP6.2, JP7.2, JP8.1, R1.1, U1.VSS@1, U1.VSS@2, U2.ADJ, X4.GND, X4.SHIELD@1, X4.SHIELD@3, X4.SHIELD@4, X5.SH@1, X5.SH@2, X5.VSS1, X5.VSS2, X6.2
- net INT: now also TP4.TP, U2.P2[11]/EINT1/I2STX_CLK; no longer JP6.5, U1.PIO0_21/CT16B1_MAT0/MOSI1
- net ISP: now also JP2.2, R3.1, U2.P2[10]/EINT0/NMI; no longer R5.1, U1.PIO0_1/CLKOUT/CT32B0_MAT2/USB_FTOGGLE-(ISP)
- net LCD_D0: now also JP3.7, JP6.7, U2.P2[0]/PWM1[1]/TXD1; no longer JP1.7, U1.PIO1_0/CT32B1_MAT0
- net LCD_D1: now also JP3.8, JP6.8, U2.P2[1]/PWM1[2]/RXD1; no longer JP1.8, U1.PIO1_1/CT32B1_MAT1
- net LCD_D2: now also JP3.9, JP6.9, U2.P2[2]/PWM1[3]/CTS1/TRACEDATA[3]; no longer JP1.9, U1.PIO1_2/CT32B1_MAT2
- net LCD_D3: now also JP3.10, JP6.10, U2.P2[3]/PWM1[4]/DCD1/TRACEDATA[2]; no longer JP1.10, U1.PIO1_3/CT32B1_MAT3
- net LCD_D4: now also JP3.11, JP6.11, U2.P2[4]/PWM1[5]/DSR1/TRACEDATA[1]; no longer JP1.11, JP8.11, U1.PIO1_4/CT32B1_CAP0
- net LCD_D5: now also JP3.12, JP6.12, U2.P2[5]/PWM1[6]/DTR1/TRACEDATA[0]; no longer JP1.12, JP8.12, U1.PIO1_5/CT32B1_CAP1
- net LCD_D6: now also JP3.13, JP6.13, U2.P2[6]/PCAP1[0]/RI1/TRACECLK; no longer JP1.13, JP8.13, U1.PIO1_6
- net LCD_D7: now also JP3.14, JP6.14, U2.P2[7]/RD2/RTS1; no longer JP1.14, JP8.14, U1.PIO1_7
- net LCD_EN: now also JP3.6, JP6.6, U2.P1[27]/CLKOUT/USB_OVRCR/CAP0[1]; no longer JP1.6, JP8.6, U1.PIO0_20/CT16B1_CAP0
- net LCD_LEDB: now also R18.2, R6.2, U2.P3[26]/STCLK/MAT0[1]/PWM1[3]; no longer R16.2, R22.2, U1.PIO1_26/CT32B0_MAT2/RXD
- net LCD_LEDB_RES: now also JP3.22, R6.1; no longer JP1.22, R22.1
- net LCD_LEDB_RES1: now also JP6.18, R18.1; no longer JP8.18, R16.1
- net LCD_LEDG: now also R10.2, R20.2, U2.P3[25]/MAT0[0]/PWM1[2]; no longer R17.2, R23.2, U1.PIO1_25/CT32B0_MAT1
- net LCD_LEDG_RES: now also JP3.21, R10.1; no longer JP1.21, R23.1
- net LCD_LEDG_RES1: now also JP6.17, R20.1; no longer JP8.17, R17.1
- net LCD_LEDR: now also R11.2, R21.2, U2.P1[18]/USB_UP_LED/PWM1[1]/CAP1[0]; no longer R18.2, R24.2, U1.PIO1_24/CT32B0_MAT0
- net LCD_LEDR_RES: now also JP3.20, R11.1; no longer JP1.20, R24.1
- net LCD_LEDR_RES1: now also JP6.16, R21.1; no longer JP8.16, R18.1
- net LCD_PSB: now also JP3.15, SJ3.2; no longer JP1.15, U1.PIO1_28/CT32B0_CAP0/SCLK
- net LCD_R/W: now also JP3.5, JP6.5, U2.P1[19]/MC0A/USB_PPWR/CAP1[1]; no longer JP1.5, JP8.5, U1.SWCLK/PIO0_10/SCK0/CT16B0_MAT2
- net LCD_RS: now also JP3.4, JP6.4, U2.P1[25]/MC1A/MAT1[1]; no longer JP1.4, JP8.4, U1.PIO0_17/RTS/CT32B0_CAP0/SCLK
- net LCD_RST: now also JP2.3, JP3.17, R4.1, S3.3, S3.4, U2.P1[31]/SCK1/AD0[5]; no longer JP1.17, U1.PIO1_27/CT32B0_MAT3/TXD
- net LCD_VO: now also C17.1, JP3.3, JP6.3, R24.2; no longer C10.1, JP1.3, R1.2
- net LCD_VOUT: now also JP3.18, SJ6.3; no longer JP1.18, U3.VDD
- net P0_22: now also U2.P0[22]/RTS1/TD1, W2.P1; no longer U1.PIO0_22/AD6/CT16B1_MAT1/MISO1, W1.P7
- net P1_10: now also U2.P1[10]/ENET_RXD1, W5.P3; no longer U1.PIO1_10, W2.P3
- net P1_14: now also U2.P1[14]/ENET_RX_ER, W5.P2; no longer U1.PIO1_14/DSR/CT16B0_MAT1/RXD, W2.P7
- net P1_15: now also U2.P1[15]/ENET_REF_CLK, W5.P1; no longer U1.PIO1_15/DCD/CT16B0_MAT2/SCK1, W2.P8
- net P1_8: now also U2.P1[8]/ENET_CRS, W5.P5; no longer U1.PIO1_8, W2.P1
- net P1_9: now also U2.P1[9]/ENET_RXD0, W5.P4; no longer U1.PIO1_9, W2.P2
- net RESET: now also JP2.1, R2.1, U2.RESET; no longer R4.1, U1.RESET/PIO0_0
- net SD_CD: now also TP5.TP, U2.P2[12]/EINT2/I2STX_WS, X4.CD, X5.SHIELD@2, X5.SHIELD@4; no longer U1.PIO1_18/CT16B1_CAP1/TXD, X4.SHIELD@2, X5.CD
- net SD_WP: now also TP6.TP, U2.P2[13]/EINT3/I2STX_SDA, X4.WP; no longer U1.PIO1_19/DTR/SSEL1, X5.WP
- net SSEL1: now also R9.1, U2.P0[6]/I2SRX_SDA/SSEL1/MAT2[0], X4.CD/DAT3, X5.CS; no longer JP5.3, U1.PIO1_23/CT16B1_MAT1/SSEL1
- net USB_CONNECT: now also R15.1, TP3.TP, U2.P2[9]/USB_CONNECT/RXD2; no longer R8.1, U1.PIO0_6/USB_CONNECT/SCK0
- net USB_CONNECT_BASE: now also R15.2, R17.1; no longer R8.2, R9.1
- net USB_CONNECT_COLLECTOR: now also R23.1; no longer R2.1
- net USB_DM: now also C19.1, R19.1, U2.P0[30]/USB_D-; no longer C4.1, R6.1, U1.USB_DM
- net USB_DP: now also C18.1, R16.1, U2.P0[29]/USB_D+; no longer C3.1, R7.1, U1.USB_DP
- net USB_VBUS: now also R22.1, TP1.TP, U2.P1[30]/VBUS/AD0[4]; no longer R10.1, U1.PIO0_3/USB_VBUS
- net VBUS: now also R22.2; no longer R10.2
- net VI2C: now also C13.1, PCB1.VCC, R13.2, R14.2; no longer C9.1, JP6.1, R11.2, R3.2
- net VIN: now also JP1.1, Z1.1; no longer JP2.1, X6.1
- net VUART: now also SJ4.2; no longer SJ1.2
Other:
- note removed: "DO NOT POPULATE"
- moved on the sheet: C1, C10, C13, C14, C15, C16, C2, C3, C4, C5, C6, C7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
